Commit message: add demo to package name

File: urdf/puppet.urdf (robot description, URDF)
Before this commit: robot puppet, 20 links, 19 joints
Links:
- link head: geometry visual mesh filename=package://trep_urdf_demo/urdf/stl/head.stl scale=0.09 0.09 0.09
- link left_femur: geometry visual mesh filename=package://trep_urdf_demo/urdf/stl/femur.stl scale=0.1167 0.1167 0.1167
- link left_humerus: geometry visual mesh filename=package://trep_urdf_demo/urdf/stl/lefthumerus.stl scale=0.105 0.105 0.105
- link left_radius: geometry visual mesh filename=package://trep_urdf_demo/urdf/stl/leftradius.stl scale=0.095 0.095 0.1
- link left_tibia: geometry visual mesh filename=package://trep_urdf_demo/urdf/stl/tibia.stl scale=0.1067 0.1067 0.1067
- link right_femur: geometry visual mesh filename=package://trep_urdf_demo/urdf/stl/femur.stl scale=0.1167 0.1167 0.1167
- link right_humerus: geometry visual mesh filename=package://trep_urdf_demo/urdf/stl/righthumerus.stl scale=0.105 0.105 0.105
- link right_radius: geometry visual mesh filename=package://trep_urdf_demo/urdf/stl/rightradius.stl scale=0.095 0.095 0.1
- link right_tibia: geometry visual mesh filename=package://trep_urdf_demo/urdf/stl/tibia.stl scale=0.1067 0.1067 0.1067
- link torso: geometry visual mesh filename=package://trep_urdf_demo/urdf/stl/torso.stl scale=0.115 0.1121 0.1088
